File: Atmega_Breadboard/atmega.kicad_sch (KiCad schematic)
At the start: 7 parts, among them J2 Conn_02x03_Row_Letter_First, SW1 SW_SPST, U1 ATmega328P-P, Y1 Crystal

Commit message: up
Parts:
- added C3, C4: 22pf, Capacitor_THT:C_Disc_D4.3mm_W1.9mm_P5.00mm, symbol Device:C
- added R2: 10k, Resistor_THT:R_Axial_DIN0207_L6.3mm_D2.5mm_P2.54mm_Vertical, symbol Device:R
- added U2: ATmega328P-P, Package_DIP:DIP-28_W7.62mm, symbol MCU_Microchip_ATmega:ATmega328P-P
- added Y2: Crystal, Crystal:Crystal_HC49-4H_Vertical, symbol Device:Crystal
Connections:
- net +5V: now also R2.1, U2.20 (AVCC), U2.21 (AREF), U2.7 (VCC)
- net GND: now also C3.2, C4.2, U2.22 (GND), U2.8 (GND)
- new net: C3.1, U2.10 (XTAL2/PB7), Y2.1
- new net: C4.1, U2.9 (XTAL1/PB6), Y2.2
- new net: R2.2, U2.1 (~{RESET}/PC6)
